File: Repeater_memris_V2a/Repeater_memris_V2a.kicad_pcb (KiCad board)
At the start: 4 copper layers, 96 x 83 mm, 73 parts, among them J2 Conn_01x06_Socket, Q1 MMBT2222A, Q2 MMBT2222A, U1 ATmega328-A, U2 AMS1117-3.3, U3 SA868-U, U4 SA868-V, U5 4016, U6 SPF5043Z, Y1 Crystal_GND2

Commit message: update
Parts:
- removed TP1, TP10, TP11, TP12, TP14, TP2, TP8, TP9: TestPoint, TestPoint:TestPoint_Loop_D1.80mm_Drill1.0mm_Beaded
- added C18: 100nF, Capacitor_SMD:C_0603_1608Metric, F.Cu at (-10.0, 135.3)
- added C30: 15pF, Spacemanic_SMD:C_0603_HS, F.Cu at (-17.4, 135.3)
- added C31: 1.8pF, Spacemanic_SMD:C_0603_HS, F.Cu at (-17.4, 137.8)
- added C32: 10pF, Spacemanic_SMD:C_0603_HS, F.Cu at (-17.4, 140.2)
- added C33: 1.8pF, Spacemanic_SMD:C_0603_HS, F.Cu at (-17.4, 142.7)
- added C34: 15pF, Spacemanic_SMD:C_0603_HS, F.Cu at (-17.4, 145.2)
- added L10: 8.2nH, Spacemanic_SMD:L_0603_HS, F.Cu at (-13.8, 140.2)
- added L11: 8.2nH, Spacemanic_SMD:L_0603_HS, F.Cu at (-13.8, 142.7)
- added L12: 22nH, Spacemanic_SMD:L_0603_HS, F.Cu at (-13.8, 145.2)
- added L8: 22nH, Spacemanic_SMD:L_0603_HS, F.Cu at (-13.8, 135.3)
- added L9: 8.2nH, Spacemanic_SMD:L_0603_HS, F.Cu at (-13.8, 137.8)
Connections:
- C14 pad 1: GND -> unconnected-(C14-Pad1)
- C14 pad 2: +5V -> unconnected-(C14-Pad2)
- C4 pad 1: GND -> unconnected-(C4-Pad1)
- C4 pad 2: +5V -> unconnected-(C4-Pad2)
- C5 pad 1: +5V -> unconnected-(C5-Pad1)
- C5 pad 2: GND -> unconnected-(C5-Pad2)
- U3 pad 12: unconnected-(U3-ANT-Pad12) -> Net-(U3-ANT)
- U6 pad 1: unconnected-(U6-Pad1) -> Net-(C19-Pad1)
- U6 pad 2: unconnected-(U6-Pad2) -> GND
- U6 pad 3: unconnected-(U6-Pad3) -> Net-(C18-Pad2)
- U6 pad 4: unconnected-(U6-Pad4) -> GND
