File: Repeater_memris_V2a/Repeater_memris_V2a.kicad_sch (KiCad schematic)
At the start: 92 parts, among them J1 Conn_Coaxial, J2 Conn_01x06_Socket, Q1 MMBT2222A, Q2 MMBT2222A, U1 ATmega328-A, U2 AMS1117-3.3, U3 SA868-U, U4 SA868-V, U5 4016, U6 SPF5043Z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

Commit message: Revert "sch pcb update"
This reverts commit 82fe7de560fbc9173e196ee1871e922f74af1bd5.
Parts:
- removed C18: 100nF, Capacitor_SMD:C_0603_1608Metric, symbol Device:C_Small
- removed C19, C21, C24: 100pF, symbol Device:C_Small
- removed C20: 10nF, symbol Device:C_Small
- removed C22: 100nF, symbol Device:C_Small
- removed C23: X, symbol Device:C_Small
- removed L1, L2, L3, L4, L5, L6, L7: L_Small, symbol Device:L_Small
- removed R24, R26: X, symbol Device:R_Small
- removed R25: 0, symbol Device:R_Small
- removed U6: SPF5043Z, Package_TO_SOT_SMD:SOT-343_SC-70-4, symbol ub1qbm_parts:SPF5043Z
- C1, C10, C11, C12, C13, C14, C15, C16, C17, C2, C3, C4, C5, C6, C7, C8, C9: symbol Device:C_Small -> Device:C
Connections:
- net +3.3REF: now also C1.2, C6.2, C7.2
- net +5V: now also C11.2, C14.2, C2.2, C3.2, C4.2, C5.1
- net GND: now also C1.1, C10.2, C11.1, C14.1, C2.1, C3.1, C4.1, C5.2, C6.1, C7.1
- net MIC_IN: now also C15.1
- net Reset: now also C8.2
- net at R5.2, U1.29 (~{RESET}/PC6): now also C8.1
- net at R20.2, U5.4: now also C16.2
- net at R15.2, U5.2: now also C15.2, C16.1
- net at R1.2, R10.1, R3.2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: now also C10.1, C9.1
- net at C9.2: now also R8.1
- net at R23.2, U5.3: now also C17.2
Other:
- moved on the sheet: C11, C12, C13, C14, C15, C16, C17, H1, H2, H3, H4, H5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
