File: Repeater_memris_V2a/Repeater_memris_V2a.kicad_sch (KiCad schematic)
At the start: 74 parts, among them J1 Conn_Coaxial, J2 Conn_01x06_Socket, Q1 MMBT2222A, Q2 MMBT2222A, U1 ATmega328-A, U2 AMS1117-3.3, U3 SA868-U, U4 SA868-V, U5 4016, Y1 Crystal_GND2

Commit message: sch pcb update
Parts:
- added C18: 100nF, Capacitor_SMD:C_0603_1608Metric, symbol Device:C_Small
- added C19, C21, C24: 100pF, symbol Device:C_Small
- added C20: 10nF, symbol Device:C_Small
- added C22: 100nF, symbol Device:C_Small
- added C23: X, symbol Device:C_Small
- added L1, L2, L3, L4, L5, L6, L7: L_Small, symbol Device:L_Small
- added R24, R26: X, symbol Device:R_Small
- added R25: 0, symbol Device:R_Small
- added U6: SPF5043Z, Package_TO_SOT_SMD:SOT-343_SC-70-4, symbol ub1qbm_parts:SPF5043Z
- C1, C10, C11, C12, C13, C14, C15, C16, C17, C2, C3, C4, C5, C6, C7, C8, C9: symbol Device:C -> Device:C_Small
Connections:
- net +3.3REF: no longer C1.2, C6.2, C7.2
- net +5V: now also C20.1, C21.1, C22.1, L2.1; no longer C11.2, C14.2, C2.2, C3.2, C4.2, C5.1
- net GND: now also C20.2, C21.2, C22.2, R24.2, R26.2, U6.2, U6.4; no longer C1.1, C10.2, C11.1, C14.1, C2.1, C3.1, C4.1, C5.2, C6.1, C7.1
- net MIC_IN: no longer C15.1
- net Reset: no longer C8.2
- net at R5.2, U1.29 (~{RESET}/PC6): no longer C8.1
- net at R20.2, U5.4: no longer C16.2
- net at R15.2, U5.2: no longer C15.2, C16.1
- net at R1.2, R10.1, R3.2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: no longer C10.1, C9.1
- net at C9.2: no longer R8.1
- net at R23.2, U5.3: no longer C17.2
- net at U3.12 (ANT): now also C23.1, C24.1
- new net: L1.1, L2.2
- new net: C19.2, R24.1, R25.1
- new net: C24.2, R25.2, R26.1
- new net: C19.1, L1.2, U6.1
Other:
- moved on the sheet: C11, C12, C13, C14, C15, C16, C17, H1, H2, H3, H4, H5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

Commit message: update
Parts:
- removed L6, L7: L_Small, symbol Device:L_Small
- removed TP1, TP10, TP11, TP12, TP14, TP2, TP8, TP9: TestPoint, TestPoint:TestPoint_Loop_D1.80mm_Drill1.0mm_Beaded, symbol Connector:TestPoint
- added C25: X, symbol Device:C_Small
- added C26, C29: 100nF, symbol Device:C_Small
- added C27: 1uF, Capacitor_SMD:C_0603_1608Metric, symbol Device:C_Small
- added C28, C35: 100pF, symbol Device:C_Small
- added C30, C34: 15pF, Spacemanic_SMD:C_0603_HS, symbol Device:C_Small
- added C31, C33: 1.8pF, Spacemanic_SMD:C_0603_HS, symbol Device:C_Small
- added C32: 10pF, Spacemanic_SMD:C_0603_HS, symbol Device:C_Small
- added C36: 22pF, Spacemanic_SMD:C_0603_HS, symbol Device:C_Small
- added C37: 4.7pF, Spacemanic_SMD:C_0603_HS, symbol Device:C_Small
- added C38: 5.6pF, Spacemanic_SMD:C_0603_HS, symbol Device:C_Small
- added C39: 3.3pF, Spacemanic_SMD:C_0603_HS, symbol Device:C_Small
- added J3: Conn_Coaxial, symbol Connector:Conn_Coaxial
- added L10, L11, L9: 8.2nH, Spacemanic_SMD:L_0603_HS, symbol Device:L_Small
- added L12, L8: 22nH, Spacemanic_SMD:L_0603_HS, symbol Device:L_Small
- C12: value 1uF -> 15pF; footprint Capacitor_SMD:C_0603_1608Metric -> Spacemanic_SMD:C_0603_HS
- L3: value L_Small -> 18nH; footprint (none) -> Spacemanic_SMD:L_0603_HS
- L4: value L_Small -> 47nH; footprint (none) -> Spacemanic_SMD:L_0603_HS
- L5: value L_Small -> 39nH; footprint (none) -> Spacemanic_SMD:L_0603_HS
Connections:
- net +3.3REF: now also C1.2, C6.2, C7.2
- net +5V: now also C11.2, C2.2, C3.2, C26.1, C27.2, C28.1, C29.1, C35.1; no longer C12.2
- net GND: now also C1.1, C10.2, C11.1, C12.2, C2.1, C3.1, C6.1, C7.1, J1.2 (Ext), C26.2, C27.1, C28.2, C29.2, C30.2, C32.2, C34.2, C35.2, C36.2, C37.2, J3.2 (Ext), L10.1, L11.1, L9.1; no longer C12.1
- net MIC_IN: now also C15.1
- net Reset: now also C8.2
- net at L3.1: now also U4.12 (ANT)
- net at L3.2: now also C12.1, L4.1, C38.1
- net at R5.2, U1.29 (~{RESET}/PC6): now also C8.1
- net at R20.2, U5.4: now also C16.2
- net at C18.1: now also C25.2, L12.2
- net at C18.2: now also U6.3
- net at J1.1 (In): now also L8.1
- net at R15.2, U5.2: now also C15.2, C16.1
- net at R1.2, R10.1, R3.2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: now also C10.1, C9.1
- net at C9.2: now also R8.1
- net at L5.1: now also L4.2, C36.1, C38.2, C39.1
- net at L5.2: now also C37.1, C39.2, J3.1 (In)
- net at R23.2, U5.3: now also C17.2
- net at C23.2: now also C25.1
- new net: C31.2, C32.1, C33.1, L10.2
- new net: C30.1, C31.1, L8.2, L9.2
- new net: C33.2, C34.1, L11.2, L12.1
Other:
- note added: "BPF filter"
- note added: "Bw: 418-488MHz G: -2dB"
- moved on the sheet: C11, J1, R12, U4
