File: MEMRICK_V2/MEMRICK_V2.kicad_sch (KiCad schematic)
At the start: 106 parts, among them J1 HDR-M-2.54_1x2, J2_5 adapter_16, J3 HDR-M-2.54, J6_4 adapter_16, J7 HDR-M-2.54, Q1 BFR93A, Q2 BFR93A, Q3 BFR93A, Q4 BFR93A, T1 TP, T10 TP, T11 TP, T12 TP, T2 TP, T3 TP, T4 TP, T5 TP, T6 TP, T7 TP, T8 TP, T9 TP, U1 AD8616ARMZ, U10 LD39050PU33R, U11 LD39050PU33R, U12 ADG619BRMZ, U13 SN74LVC1T45DBVRG4, U14 SN74LVC1T45DBVRG4, U15 SN74LVC1T45DBVRG4, U2 AD8616ARMZ, U3 ADG436BRZ, U4 ADG1408YRUZ, U5 DPU01L-5, U6 ADG1408YRUZ, U7 ADG1408YRUZ, U8 ADG1408YRUZ, U9 STM32G431CBT6, X1 24.000MHz

Commit message: update
Parts:
- added U16: ADG1408YRUZ, Package_SO:TSSOP-16_4.4x5mm_P0.65mm, symbol ADG1408YRUZ-REEL7_3
- added U17, U18: ADG1408YRUZ, Package_SO:TSSOP-16_4.4x5mm_P0.65mm, symbol Analog_Switch:ADG1408YRUZ
- added U19: STM32G431CBTx, Package_QFP:LQFP-48_7x7mm_P0.5mm, symbol MCU_ST_STM32G4:STM32G431CBTx
Connections:
- new net: U19.23 (VSS), U19.35 (VSS), U19.47 (VSS)
